File: BinaryGame.kicad_pcb (KiCad board)
At the start: 2 copper layers, 85.5 x 54 mm, 45 parts, among them SW1 SW_SPST, SW10 SW_SPST, SW11 SW_SPST, SW12 SW_SPST, SW13 SW_SPST, SW14 SW_SPST, SW15 SW_SPST, SW16 SW_SPST, SW17 SW_SPST, SW18 SW_SPST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

Commit message: Update BinaryGame.kicad_pcb
Parts:
- moved SW18 1.00 mm to (181.5, 118.0)
Other:
- board text added: "Reset binary"
Changed lines of the file:
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@@
   )
   (footprint "Button_Switch_SMD:SW_SPST_CK_RS282G05A3" (layer "F.Cu")
-    (at 181.5 119)
+    (at 181.5 118)
     (descr "https://www.mouser.com/ds/2/60/RS-282G05A-SM_RT-1159762.pdf")
     (tags "SPST button tactile switch")
@@
     (effects (font (size 1.5 1.5) (thickness 0.2)))
   )
-  (gr_text "Enter result" (at 181.4 115.4) (layer "F.SilkS")
+  (gr_text "Enter result" (at 181.4 114.5) (layer "F.SilkS")
     (effects (font (size 1.5 1.5) (thickness 0.2)))
   )
@@
     (effects (font (size 1.5 1.5) (thickness 0.2)))
   )
+  (gr_text "Reset binary" (at 181.5 121.5) (layer "F.SilkS")
+    (effects (font (size 1.5 1.5) (thickness 0.2) italic))
+  )
   (gr_text "Bin to\ndecimal" (at 162.4 72.1) (layer "F.SilkS")
-    (effects (font (size 1 1) (thickness 0.15)))
+    (effects (font (size 1 1) (thickness 0.15) italic))
   )
   (gr_text "Mode" (at 155 74.4) (layer "F.SilkS")
@@
   )
   (gr_text "Bin to\nhex" (at 162.5 82.9) (layer "F.SilkS")
-    (effects (font (size 1 1) (thickness 0.15)))
+    (effects (font (size 1 1) (thickness 0.15) italic))
   )
   (gr_text "0" (at 162.5 108) (layer "F.SilkS")
